Commit message: added camera virtual frames

File: urdf/markhor.xacro (robot description, xacro)
@@ -103,4 +103,16 @@
     <xacro:property name="joint_track_rr_velocity_limit" value="5.34" />
     <xacro:property name="joint_track_rr_torque_limit" value="94.5" />
+    <!-- Front Camera -->
+    <xacro:property name="joint_front_cam" value="front_cam" />
+    <xacro:property name="joint_front_cam_type" value="fixed" />
+    <xacro:property name="joint_front_cam_axis_xyz" value="0 0 0" />
+    <xacro:property name="joint_front_cam_origin_xyz" value="0.35864800 0 -0.03810000" />
+    <xacro:property name="joint_front_cam_origin_rpy" value="0 ${pi/2} 0" />
+    <!-- Rear Camera -->
+    <xacro:property name="joint_rear_cam" value="rear_cam" />
+    <xacro:property name="joint_rear_cam_type" value="fixed" />
+    <xacro:property name="joint_rear_cam_axis_xyz" value="0 0 0" />
+    <xacro:property name="joint_rear_cam_origin_xyz" value="-0.35864800 0 -0.03810000" />
+    <xacro:property name="joint_rear_cam_origin_rpy" value="0 ${-pi/2} 0" />
     <!-- Anchor for a robotic arm -->
     <xacro:property name="joint_arm_root" value="arm_root" />
@@ -129,4 +141,10 @@
         <xacro:kinova_link link_name="${prefix}_link_flip_rr" link_mesh="${link_flip_rr_mesh}"/>
         <xacro:kinova_joint joint_name="${prefix}_joint_flip_rr" type="${joint_flip_rr_type}" parent="${prefix}_link_gb_rr" child="${prefix}_link_flip_rr" joint_axis_xyz="${joint_flip_rr_axis_xyz}" joint_origin_xyz="${joint_flip_rr_origin_xyz}" joint_origin_rpy="${joint_flip_rr_origin_rpy}" joint_lower_limit="${joint_flip_rr_lower_limit}" joint_upper_limit="${joint_flip_rr_upper_limit}" joint_velocity_limit="${joint_flip_rr_velocity_limit}" joint_torque_limit="${joint_flip_rr_torque_limit}"/>
+        <!-- Anchor for the front camera -->
+        <xacro:kinova_virtual_link link_name="${prefix}_link_front_cam"/>
+        <xacro:kinova_virtual_joint joint_name="${prefix}_joint_front_cam" type="${joint_front_cam_type}" parent="${prefix}_link_base" child="${prefix}_link_front_cam" joint_axis_xyz="${joint_front_cam_axis_xyz}" joint_origin_xyz="${joint_front_cam_origin_xyz}" joint_origin_rpy="${joint_front_cam_origin_rpy}" joint_lower_limit="0" joint_upper_limit="0"/>
+        <!-- Anchor for the rear camera -->
+        <xacro:kinova_virtual_link link_name="${prefix}_link_rear_cam"/>
+        <xacro:kinova_virtual_joint joint_name="${prefix}_joint_rear_cam" type="${joint_rear_cam_type}" parent="${prefix}_link_base" child="${prefix}_link_rear_cam" joint_axis_xyz="${joint_rear_cam_axis_xyz}" joint_origin_xyz="${joint_rear_cam_origin_xyz}" joint_origin_rpy="${joint_rear_cam_origin_rpy}" joint_lower_limit="0" joint_upper_limit="0"/>
         <!-- Anchor for a robotic arm -->
         <xacro:kinova_virtual_link link_name="${prefix}_link_arm_root"/>

Commit message: wip added ovis and sick lidar

File: urdf/markhor.xacro (robot description, xacro)
@@ -121,4 +121,10 @@
     <xacro:property name="joint_arm_root_origin_xyz" value="0.17394875 0 -0.12291060" />
     <xacro:property name="joint_arm_root_origin_rpy" value="${pi} 0 0" />
+    <!-- LiDAR -->
+    <xacro:property name="joint_lidar" value="lidar" />
+    <xacro:property name="joint_lidar_type" value="fixed" />
+    <xacro:property name="joint_lidar_axis_xyz" value="0 0 0" />
+    <xacro:property name="joint_lidar_origin_xyz" value="0.32034017 0 -0.1393156" />
+    <xacro:property name="joint_lidar_origin_rpy" value="${pi} 0 0" />
     <xacro:macro name="markhor" params="base_parent prefix:=markhor">
         <xacro:kinova_link link_name="${prefix}_link_base" link_mesh="${link_base_mesh}" link_origin_rpy="${link_base_origin_rpy}"/>
@@ -150,4 +156,7 @@
         <xacro:kinova_virtual_link link_name="${prefix}_link_arm_root"/>
         <xacro:kinova_virtual_joint joint_name="${prefix}_joint_arm_root" type="${joint_arm_root_type}" parent="${prefix}_link_base" child="${prefix}_link_arm_root" joint_axis_xyz="${joint_arm_root_axis_xyz}" joint_origin_xyz="${joint_arm_root_origin_xyz}" joint_origin_rpy="${joint_arm_root_origin_rpy}" joint_lower_limit="0" joint_upper_limit="0"/>
+        <!-- Anchor for the LiDAR -->
+        <xacro:kinova_virtual_link link_name="${prefix}_link_lidar"/>
+        <xacro:kinova_virtual_joint joint_name="${prefix}_joint_lidar" type="${joint_lidar_type}" parent="${prefix}_link_base" child="${prefix}_link_lidar" joint_axis_xyz="${joint_lidar_axis_xyz}" joint_origin_xyz="${joint_lidar_origin_xyz}" joint_origin_rpy="${joint_lidar_origin_rpy}" joint_lower_limit="0" joint_upper_limit="0"/>
     </xacro:macro>
 </root>

File: urdf/markhor_standalone.xacro (robot description, xacro)
@@ -3,6 +3,6 @@
   <!-- Include markhor robot -->
   <xacro:include filename="$(find markhor_description)/urdf/markhor.xacro"/>
-  <link name="root"/>
-  <xacro:property name="robot_root" value="root" />
+  <link name="markhor_root"/>
+  <xacro:property name="robot_root" value="markhor_root" />
   <xacro:markhor base_parent="${robot_root}"/>
 </robot>
