Commit message: added link materials (colors)

File: urdf/kinova_common.xacro (robot description, xacro)
@@ -14,5 +14,6 @@
   xmlns:physics="http://playerstage.sourceforge.net/gazebo/xmlschema/#physics"
   xmlns:xacro="http://www.ros.org/wiki/xacro">
-  <xacro:macro name="kinova_link" params="link_name link_mesh link_origin_xyz:='0 0 0' link_origin_rpy:='0 0 0' has_collision_mesh:=false">
+  <xacro:include filename="$(find markhor_description)/urdf/materials.xacro"/>
+  <xacro:macro name="kinova_link" params="link_name link_mesh link_origin_xyz:='0 0 0' link_origin_rpy:='0 0 0' link_material:='red' has_collision_mesh:=false">
     <link name="${link_name}">
       <visual>
@@ -21,4 +22,5 @@
         </geometry>
         <origin xyz="${link_origin_xyz}" rpy="${link_origin_rpy}"/>
+        <material name="${link_material}"/>
       </visual>
       <collision>

File: urdf/markhor.xacro (robot description, xacro)
@@ -10,8 +10,10 @@
     <xacro:property name="link_gb_rl_mesh" value="mk_gb_fr"/>
     <xacro:property name="link_gb_rr_mesh" value="mk_gb_fl"/>
+    <xacro:property name="link_gb_material" value="grey"/>
     <xacro:property name="link_flip_fl_mesh" value="mk_flip"/>
     <xacro:property name="link_flip_fr_mesh" value="mk_flip"/>
     <xacro:property name="link_flip_rl_mesh" value="mk_flip"/>
     <xacro:property name="link_flip_rr_mesh" value="mk_flip"/>
+    <xacro:property name="link_flip_material" value="black"/>
     <xacro:property name="joint_base" value="joint_base"/>
     <xacro:property name="joint_base_type" value="fixed"/>
@@ -130,20 +132,20 @@
         <xacro:kinova_link link_name="${prefix}_link_base" link_mesh="${link_base_mesh}" link_origin_rpy="${link_base_origin_rpy}"/>
         <xacro:kinova_joint joint_name="${prefix}_joint_base" type="${joint_base_type}" parent="${base_parent}" child="${prefix}_link_base" joint_axis_xyz="${joint_base_axis_xyz}" joint_origin_xyz="${joint_base_origin_xyz}" joint_origin_rpy="${joint_base_origin_rpy}" joint_lower_limit="0" joint_upper_limit="0" joint_velocity_limit="0" joint_torque_limit="0" fixed="true"/>
-        <xacro:kinova_link link_name="${prefix}_link_gb_fl" link_mesh="${link_gb_fl_mesh}" />
+        <xacro:kinova_link link_name="${prefix}_link_gb_fl" link_mesh="${link_gb_fl_mesh}" link_material="${link_gb_material}"/>
         <xacro:kinova_joint joint_name="${prefix}_joint_gb_fl" type="${joint_gb_fl_type}" parent="${prefix}_link_base" child="${prefix}_link_gb_fl" joint_axis_xyz="${joint_gb_fl_axis_xyz}" joint_origin_xyz="${joint_gb_fl_origin_xyz}" joint_origin_rpy="${joint_gb_fl_origin_rpy}" joint_lower_limit="0" joint_upper_limit="0" joint_velocity_limit="0" joint_torque_limit="0" fixed="true"/>
-        <xacro:kinova_link link_name="${prefix}_link_gb_fr" link_mesh="${link_gb_fr_mesh}" link_origin_rpy="${link_gb_fr_origin_rpy}"/>
+        <xacro:kinova_link link_name="${prefix}_link_gb_fr" link_mesh="${link_gb_fr_mesh}" link_origin_rpy="${link_gb_fr_origin_rpy}" link_material="${link_gb_material}"/>
         <xacro:kinova_joint joint_name="${prefix}_joint_gb_fr" type="${joint_gb_fr_type}" parent="${prefix}_link_base" child="${prefix}_link_gb_fr" joint_axis_xyz="${joint_gb_fr_axis_xyz}" joint_origin_xyz="${joint_gb_fr_origin_xyz}" joint_origin_rpy="${joint_gb_fr_origin_rpy}" joint_lower_limit="0" joint_upper_limit="0" joint_velocity_limit="0" joint_torque_limit="0" fixed="true"/>
-        <xacro:kinova_link link_name="${prefix}_link_gb_rl" link_mesh="${link_gb_rl_mesh}" />
+        <xacro:kinova_link link_name="${prefix}_link_gb_rl" link_mesh="${link_gb_rl_mesh}" link_material="${link_gb_material}"/>
         <xacro:kinova_joint joint_name="${prefix}_joint_gb_rl" type="${joint_gb_rl_type}" parent="${prefix}_link_base" child="${prefix}_link_gb_rl" joint_axis_xyz="${joint_gb_rl_axis_xyz}" joint_origin_xyz="${joint_gb_rl_origin_xyz}" joint_origin_rpy="${joint_gb_rl_origin_rpy}" joint_lower_limit="0" joint_upper_limit="0" joint_velocity_limit="0" joint_torque_limit="0" fixed="true"/>
-        <xacro:kinova_link link_name="${prefix}_link_gb_rr" link_mesh="${link_gb_rr_mesh}" />
+        <xacro:kinova_link link_name="${prefix}_link_gb_rr" link_mesh="${link_gb_rr_mesh}" link_material="${link_gb_material}"/>
         <xacro:kinova_joint joint_name="${prefix}_joint_gb_rr" type="${joint_gb_rr_type}" parent="${prefix}_link_base" child="${prefix}_link_gb_rr" joint_axis_xyz="${joint_gb_rr_axis_xyz}" joint_origin_xyz="${joint_gb_rr_origin_xyz}" joint_origin_rpy="${joint_gb_rr_origin_rpy}" joint_lower_limit="0" joint_upper_limit="0" joint_velocity_limit="0" joint_torque_limit="0" fixed="true"/>
         <!-- flipper angle frame -->
-        <xacro:kinova_link link_name="${prefix}_link_flip_fl" link_mesh="${link_flip_fl_mesh}"/>
+        <xacro:kinova_link link_name="${prefix}_link_flip_fl" link_mesh="${link_flip_fl_mesh}" link_material="${link_flip_material}"/>
         <xacro:kinova_joint joint_name="${prefix}_joint_flip_fl" type="${joint_flip_fl_type}" parent="${prefix}_link_gb_fl" child="${prefix}_link_flip_fl" joint_axis_xyz="${joint_flip_fl_axis_xyz}" joint_origin_xyz="${joint_flip_fl_origin_xyz}" joint_origin_rpy="${joint_flip_fl_origin_rpy}" joint_lower_limit="${joint_flip_fl_lower_limit}" joint_upper_limit="${joint_flip_fl_upper_limit}" joint_velocity_limit="${joint_flip_fl_velocity_limit}" joint_torque_limit="${joint_flip_fl_torque_limit}"/>
-        <xacro:kinova_link link_name="${prefix}_link_flip_fr" link_mesh="${link_flip_fr_mesh}"/>
+        <xacro:kinova_link link_name="${prefix}_link_flip_fr" link_mesh="${link_flip_fr_mesh}" link_material="${link_flip_material}"/>
         <xacro:kinova_joint joint_name="${prefix}_joint_flip_fr" type="${joint_flip_fr_type}" parent="${prefix}_link_gb_fr" child="${prefix}_link_flip_fr" joint_axis_xyz="${joint_flip_fr_axis_xyz}" joint_origin_xyz="${joint_flip_fr_origin_xyz}" joint_origin_rpy="${joint_flip_fr_origin_rpy}" joint_lower_limit="${joint_flip_fr_lower_limit}" joint_upper_limit="${joint_flip_fr_upper_limit}" joint_velocity_limit="${joint_flip_fr_velocity_limit}" joint_torque_limit="${joint_flip_fr_torque_limit}"/>
-        <xacro:kinova_link link_name="${prefix}_link_flip_rl" link_mesh="${link_flip_rl_mesh}"/>
+        <xacro:kinova_link link_name="${prefix}_link_flip_rl" link_mesh="${link_flip_rl_mesh}" link_material="${link_flip_material}"/>
         <xacro:kinova_joint joint_name="${prefix}_joint_flip_rl" type="${joint_flip_rl_type}" parent="${prefix}_link_gb_rl" child="${prefix}_link_flip_rl" joint_axis_xyz="${joint_flip_rl_axis_xyz}" joint_origin_xyz="${joint_flip_rl_origin_xyz}" joint_origin_rpy="${joint_flip_rl_origin_rpy}" joint_lower_limit="${joint_flip_rl_lower_limit}" joint_upper_limit="${joint_flip_rl_upper_limit}" joint_velocity_limit="${joint_flip_rl_velocity_limit}" joint_torque_limit="${joint_flip_rl_torque_limit}"/>
-        <xacro:kinova_link link_name="${prefix}_link_flip_rr" link_mesh="${link_flip_rr_mesh}"/>
+        <xacro:kinova_link link_name="${prefix}_link_flip_rr" link_mesh="${link_flip_rr_mesh}" link_material="${link_flip_material}"/>
         <xacro:kinova_joint joint_name="${prefix}_joint_flip_rr" type="${joint_flip_rr_type}" parent="${prefix}_link_gb_rr" child="${prefix}_link_flip_rr" joint_axis_xyz="${joint_flip_rr_axis_xyz}" joint_origin_xyz="${joint_flip_rr_origin_xyz}" joint_origin_rpy="${joint_flip_rr_origin_rpy}" joint_lower_limit="${joint_flip_rr_lower_limit}" joint_upper_limit="${joint_flip_rr_upper_limit}" joint_velocity_limit="${joint_flip_rr_velocity_limit}" joint_torque_limit="${joint_flip_rr_torque_limit}"/>
         <!-- Anchor for the front camera -->

Commit message: adding IMU

File: urdf/kinova_common.xacro (robot description, xacro)
@@ -16,5 +16,5 @@
   <xacro:include filename="$(find markhor_description)/urdf/markhor_inertial.xacro" />
   <xacro:include filename="$(find markhor_description)/urdf/materials.xacro"/>
-  <xacro:macro name="kinova_link" params="link_name link_mesh link_origin_xyz:='0 0 0' link_origin_rpy:='0 0 0' link_material:='red' has_collision_mesh:=false">
+  <xacro:macro name="kinova_link" params="link_name link_mesh link_origin_xyz:='0 0 0' link_origin_rpy:='0 0 0' link_material:='Red' has_collision_mesh:=false">
     <link name="${link_name}">
       <visual>
@@ -24,4 +24,7 @@
         <origin xyz="${link_origin_xyz}" rpy="${link_origin_rpy}"/>
         <material name="${link_material}"/>
+        <gazebo reference="${link_name}">
+          <material>Gazebo/${link_material}</material>
+        </gazebo>
       </visual>
       <collision>

File: urdf/markhor.xacro (robot description, xacro)
@@ -10,10 +10,10 @@
     <xacro:property name="link_gb_rl_mesh" value="mk_gb_fr"/>
     <xacro:property name="link_gb_rr_mesh" value="mk_gb_fl"/>
-    <xacro:property name="link_gb_material" value="grey"/>
+    <xacro:property name="link_gb_material" value="Grey"/>
     <xacro:property name="link_flip_fl_mesh" value="mk_flip"/>
     <xacro:property name="link_flip_fr_mesh" value="mk_flip"/>
     <xacro:property name="link_flip_rl_mesh" value="mk_flip"/>
     <xacro:property name="link_flip_rr_mesh" value="mk_flip"/>
-    <xacro:property name="link_flip_material" value="black"/>
+    <xacro:property name="link_flip_material" value="Black"/>
     <xacro:property name="joint_base" value="joint_base"/>
     <xacro:property name="joint_base_type" value="fixed"/>

File: urdf/markhor_w_attachments.xacro (robot description, xacro)
@@ -25,3 +25,6 @@
   <xacro:property name="joint_fix_lidar_origin_rpy" value="0 0 0" />
   <xacro:kinova_virtual_joint joint_name="markhor_joint_fix_lidar" type="${joint_fix_lidar_type}" parent="markhor_link_lidar" child="laser_mount_link" joint_axis_xyz="${joint_fix_lidar_axis_xyz}" joint_origin_xyz="${joint_fix_lidar_origin_xyz}" joint_origin_rpy="${joint_fix_lidar_origin_rpy}" joint_lower_limit="0" joint_upper_limit="0"/>
+  <!-- IMU -->
+  <xacro:include filename="$(find markhor_description)/urdf/sensors.xacro"/>
+  <xacro:IMU robot_name="markhor" parent="markhor_link_base"/>
 </robot>

File: urdf/materials.xacro (robot description, xacro)
@@ -12,26 +12,26 @@
   xmlns:physics="http://playerstage.sourceforge.net/gazebo/xmlschema/#physics"
   xmlns:xacro="http://www.ros.org/wiki/xacro">
-<material name="black">
+<material name="Black">
   <color rgba="0.0 0.0 0.0 1.0"/>
 </material>
-<material name="blue">
+<material name="Blue">
   <color rgba="0.0 0.0 0.8 1.0"/>
 </material>
-<material name="green">
+<material name="Green">
   <color rgba="0.0 0.8 0.0 1.0"/>
 </material>
-<material name="grey">
+<material name="Grey">
   <color rgba="0.2 0.2 0.2 1.0"/>
 </material>
-<material name="orange">
+<material name="Orange">
   <color rgba="${255/255} ${108/255} ${10/255} 1.0"/>
 </material>
-<material name="brown">
+<material name="Brown">
   <color rgba="${222/255} ${207/255} ${195/255} 1.0"/>
 </material>
-<material name="red">
+<material name="Red">
   <color rgba="0.8 0.0 0.0 1.0"/>
 </material>
-<material name="white">
+<material name="White">
   <color rgba="1.0 1.0 1.0 1.0"/>
 </material>

Commit message: added sim wheels

File: urdf/kinova_common.xacro (robot description, xacro)
@@ -84,3 +84,19 @@
     </joint>
   </xacro:macro>
+  <xacro:macro name="sim_wheel" params="wheel_name wheel_rad wheel_width wheel_parent">
+    <link name="${wheel_name}_link">
+      <visual>
+        <geometry>
+          <cylinder length="${wheel_width}" radius="${wheel_rad}"/>
+        </geometry>
+        <origin xyz="0 0 0" rpy="0 ${pi/2} 0"/>
+        <material name="white"/>
+      </visual>
+    </link>
+    <joint name="${wheel_name}_joint" type="continuous">
+      <parent link="${wheel_parent}"/>
+      <child link="${wheel_name}_link"/>
+      <axis xyz="1 0 0"/>
+    </joint>
+  </xacro:macro>
 </root>

File: urdf/markhor.xacro (robot description, xacro)
@@ -129,4 +129,20 @@
     <xacro:property name="joint_lidar_origin_xyz" value="0.32034017 0 -0.1393156" />
     <xacro:property name="joint_lidar_origin_rpy" value="${pi} 0 0" />
+    <!-- FL Wheel -->
+    <xacro:property name="fl_wheel_name" value="fl_wheel"/>
+    <xacro:property name="fl_wheel_rad" value="0.1318"/>
+    <xacro:property name="fl_wheel_width" value="0.12065"/>
+    <!-- FR Wheel -->
+    <xacro:property name="fr_wheel_name" value="fr_wheel"/>
+    <xacro:property name="fr_wheel_rad" value="0.1318"/>
+    <xacro:property name="fr_wheel_width" value="0.12065"/>
+    <!-- RL Wheel -->
+    <xacro:property name="rl_wheel_name" value="rl_wheel"/>
+    <xacro:property name="rl_wheel_rad" value="0.1318"/>
+    <xacro:property name="rl_wheel_width" value="0.12065"/>
+    <!-- RR Wheel -->
+    <xacro:property name="rr_wheel_name" value="rr_wheel"/>
+    <xacro:property name="rr_wheel_rad" value="0.1318"/>
+    <xacro:property name="rr_wheel_width" value="0.12065"/>
     <xacro:macro name="markhor" params="base_parent prefix:=markhor">
         <xacro:kinova_link link_name="${prefix}_link_base" link_mesh="${link_base_mesh}" link_origin_rpy="${link_base_origin_rpy}"/>
@@ -161,4 +177,12 @@
         <xacro:kinova_virtual_link link_name="${prefix}_link_lidar"/>
         <xacro:kinova_virtual_joint joint_name="${prefix}_joint_lidar" type="${joint_lidar_type}" parent="${prefix}_link_base" child="${prefix}_link_lidar" joint_axis_xyz="${joint_lidar_axis_xyz}" joint_origin_xyz="${joint_lidar_origin_xyz}" joint_origin_rpy="${joint_lidar_origin_rpy}" joint_lower_limit="0" joint_upper_limit="0"/>
+        <!-- FL Wheel -->
+        <xacro:sim_wheel wheel_name="${fl_wheel_name}" wheel_rad="${fl_wheel_rad}" wheel_width="${fl_wheel_width}" wheel_parent="${prefix}_link_flip_fl"/>
+        <!-- FR Wheel -->
+        <xacro:sim_wheel wheel_name="${fr_wheel_name}" wheel_rad="${fr_wheel_rad}" wheel_width="${fr_wheel_width}" wheel_parent="${prefix}_link_flip_fr"/>
+        <!-- RL Wheel -->
+        <xacro:sim_wheel wheel_name="${rl_wheel_name}" wheel_rad="${rl_wheel_rad}" wheel_width="${rl_wheel_width}" wheel_parent="${prefix}_link_flip_rl"/>
+        <!-- RR Wheel -->
+        <xacro:sim_wheel wheel_name="${rr_wheel_name}" wheel_rad="${rr_wheel_rad}" wheel_width="${rr_wheel_width}" wheel_parent="${prefix}_link_flip_rr"/>
     </xacro:macro>
 </root>
