Commit message: fixed inertia parameters.

File: urdf/markhor_inertial.xacro (robot description, xacro)
@@ -25,7 +25,7 @@
         <xacro:if value="${link_name == 'markhor_link_gb_fl'}">
             <inertial>
-                <mass value="0.7477"/>
-                <origin xyz="0 -0.002 -0.0605" rpy="0 0 0"/>
-                <inertia ixx="0.385006414" ixy="0.0000696244868" ixz="-0.000181517937" iyy="0.624959190" iyz="0.000000162897534" izz="0.798949961"/>
+                <mass value="2.5"/>
+                <origin xyz="0.038 -0.038 0.014" rpy="0 0 0"/>
+                <inertia ixx="6.06448598e-2" ixy="1.93186915e-4" ixz="-1.57873663e-5" iyy="1.82869143e-2" iyz="2.81755463e-3" izz="5.13408129e-2"/>
             </inertial>
         </xacro:if>
@@ -33,7 +33,7 @@
         <xacro:if value="${link_name == 'markhor_link_gb_fr'}">
             <inertial>
-                <mass value="0.7477"/>
-                <origin xyz="0 -0.002 -0.0605" rpy="0 0 0"/>
-                <inertia ixx="0.385006414" ixy="0.0000696244868" ixz="-0.000181517937" iyy="0.624959190" iyz="0.000000162897534" izz="0.798949961"/>
+                <mass value="2.5"/>
+                <origin xyz="-0.038 -0.038 0.014" rpy="0 0 0"/>
+                <inertia ixx="6.06448598e-2" ixy="-1.93186915e-4" ixz="1.57873663e-5" iyy="1.82869143e-2" iyz="2.81755463e-3" izz="5.13408129e-2"/>
             </inertial>
         </xacro:if>
@@ -41,7 +41,7 @@
         <xacro:if value="${link_name == 'markhor_link_gb_rl'}">
             <inertial>
-                <mass value="0.7477"/>
-                <origin xyz="0 -0.002 -0.0605" rpy="0 0 0"/>
-                <inertia ixx="0.385006414" ixy="0.0000696244868" ixz="-0.000181517937" iyy="0.624959190" iyz="0.000000162897534" izz="0.798949961"/>
+                <mass value="2.5"/>
+                <origin xyz="-0.038 -0.038 0.014" rpy="0 0 0"/>
+                <inertia ixx="6.06448598e-2" ixy="-1.93186915e-4" ixz="1.57873663e-5" iyy="1.82869143e-2" iyz="2.81755463e-3" izz="5.13408129e-2"/>
             </inertial>
         </xacro:if>
@@ -49,7 +49,7 @@
         <xacro:if value="${link_name == 'markhor_link_gb_rr'}">
             <inertial>
-                <mass value="0.7477"/>
-                <origin xyz="0 -0.002 -0.0605" rpy="0 0 0"/>
-                <inertia ixx="0.385006414" ixy="0.0000696244868" ixz="-0.000181517937" iyy="0.624959190" iyz="0.000000162897534" izz="0.798949961"/>
+                <mass value="2.5"/>
+                <origin xyz="0.038 -0.038 0.014" rpy="0 0 0"/>
+                <inertia ixx="6.06448598e-2" ixy="1.93186915e-4" ixz="-1.57873663e-5" iyy="1.82869143e-2" iyz="2.81755463e-3" izz="5.13408129e-2"/>
             </inertial>
         </xacro:if>
@@ -57,7 +57,7 @@
         <xacro:if value="${link_name == 'markhor_link_flip_fl'}">
             <inertial>
-                <mass value="0.7477"/>
-                <origin xyz="0 -0.002 -0.0605" rpy="0 0 0"/>
-                <inertia ixx="0.385006414" ixy="0.0000696244868" ixz="-0.000181517937" iyy="0.624959190" iyz="0.000000162897534" izz="0.798949961"/>
+                <mass value="6.9"/>
+                <origin xyz="0 0.116 0" rpy="0 0 0"/>
+                <inertia ixx="0.268046334" ixy="0.000960466048" ixz="0.000262590776" iyy="0.0573569235" iyz="0.0000904647719" izz="0.232597105"/>
             </inertial>
         </xacro:if>
@@ -65,7 +65,7 @@
         <xacro:if value="${link_name == 'markhor_link_flip_fr'}">
             <inertial>
-                <mass value="0.7477"/>
-                <origin xyz="0 -0.002 -0.0605" rpy="0 0 0"/>
-                <inertia ixx="0.385006414" ixy="0.0000696244868" ixz="-0.000181517937" iyy="0.624959190" iyz="0.000000162897534" izz="0.798949961"/>
+                <mass value="6.9"/>
+                <origin xyz="0 0.116 0" rpy="0 0 0"/>
+                <inertia ixx="0.268046334" ixy="0.000960466048" ixz="0.000262590776" iyy="0.0573569235" iyz="0.0000904647719" izz="0.232597105"/>
             </inertial>
         </xacro:if>
@@ -73,7 +73,7 @@
         <xacro:if value="${link_name == 'markhor_link_flip_rl'}">
             <inertial>
-                <mass value="0.7477"/>
-                <origin xyz="0 -0.002 -0.0605" rpy="0 0 0"/>
-                <inertia ixx="0.385006414" ixy="0.0000696244868" ixz="-0.000181517937" iyy="0.624959190" iyz="0.000000162897534" izz="0.798949961"/>
+                <mass value="6.9"/>
+                <origin xyz="0 0.116 0" rpy="0 0 0"/>
+                <inertia ixx="0.268046334" ixy="0.000960466048" ixz="0.000262590776" iyy="0.0573569235" iyz="0.0000904647719" izz="0.232597105"/>
             </inertial>
         </xacro:if>
@@ -81,7 +81,7 @@
         <xacro:if value="${link_name == 'markhor_link_flip_rr'}">
             <inertial>
-                <mass value="0.7477"/>
-                <origin xyz="0 -0.002 -0.0605" rpy="0 0 0"/>
-                <inertia ixx="0.385006414" ixy="0.0000696244868" ixz="-0.000181517937" iyy="0.624959190" iyz="0.000000162897534" izz="0.798949961"/>
+                <mass value="6.9"/>
+                <origin xyz="0 0.116 0" rpy="0 0 0"/>
+                <inertia ixx="0.268046334" ixy="0.000960466048" ixz="0.000262590776" iyy="0.0573569235" iyz="0.0000904647719" izz="0.232597105"/>
             </inertial>
         </xacro:if>
